File: diyBMS-Leaf.kicad_pcb (KiCad board)
At the start: 2 copper layers, 218 x 30 mm, 72 parts, among them J1 AVR-ISP-6, J2 B4B-PH-K(LF)(SN), J3 AVR-ISP-6, J4 Conn_01x02, J5 Conn_01x02, Q1 IRLML6244TRPBF, Q2 IRLML6244TRPBF, U1 ATtiny841-SSU, U2 EL3H7(B)(TA)-G, U3 ATtiny841-SSU, U4 EL3H7(B)(TA)-G

Commit message: Updated with latest (#3)
* Updated with latest

* V2.0.1
Parts:
- removed C2, C5: 2.2uF, Capacitor_SMD:C_0805_2012Metric_Pad1.15x1.40mm_HandSolder
- removed C3, C6: 10uF 10V, Capacitor_SMD:C_0805_2012Metric_Pad1.15x1.40mm_HandSolder
- removed C4: 100nF, Capacitor_SMD:C_0805_2012Metric_Pad1.15x1.40mm_HandSolder
- removed D2, D6: Green, LED_SMD:LED_0805_2012Metric_Pad1.15x1.40mm_HandSolder
- removed D5: AZ432ANTR-E1, Package_TO_SOT_SMD:SOT-23
- removed D7: Blue, LED_SMD:LED_0805_2012Metric_Pad1.15x1.40mm_HandSolder
- removed D8: RED LED, LED_SMD:LED_0805_2012Metric_Pad1.15x1.40mm_HandSolder
- removed J1, J3: AVR-ISP-6, Connector_PinHeader_2.54mm:PinHeader_2x03_P2.54mm_Vertical
- removed J2: B4B-PH-K(LF)(SN), Connector_JST:JST_PH_B4B-PH-K_1x04_P2.00mm_Vertical
- removed J4, J5: Conn_01x02, Connector_PinHeader_2.54mm:PinHeader_1x02_P2.54mm_Vertical
- removed Q2: IRLML6244TRPBF, Package_TO_SOT_SMD:SOT-23
- removed R10, R32: 4K7, Resistor_SMD:R_0805_2012Metric_Pad1.15x1.40mm_HandSolder
- removed R11, R12, R14, R15, R16, R17, R20, R21: 33R, Resistor_SMD:R_2512_6332Metric_Pad1.52x3.35mm_HandSolder
- removed R18, R35, R40: 510R, Resistor_SMD:R_0805_2012Metric_Pad1.15x1.40mm_HandSolder
- removed R23: 10K, Resistor_SMD:R_0805_2012Metric_Pad1.15x1.40mm_HandSolder
- removed R24: NCP21WB473J03RA, Resistors_SMD:R_0603_HandSoldering
- removed R25, R29, R41, R7: 47K, Resistor_SMD:R_0805_2012Metric_Pad1.15x1.40mm_HandSolder
- removed R26: 1K, Resistor_SMD:R_0805_2012Metric_Pad1.15x1.40mm_HandSolder
- removed R27: 68K, Resistor_SMD:R_0805_2012Metric_Pad1.15x1.40mm_HandSolder
- removed R28: 27K, Resistor_SMD:R_0805_2012Metric_Pad1.15x1.40mm_HandSolder
- removed R30, R31, R44, R8: 2K2, Resistor_SMD:R_0805_2012Metric_Pad1.15x1.40mm_HandSolder
- removed R33, R34, R36, R37, R38, R39, R42, R43: 31R6, Resistor_SMD:R_2512_6332Metric_Pad1.52x3.35mm_HandSolder
- removed RX2: B2B-PH-K(LF)(SN), Connector_JST:JST_PH_B2B-PH-K_1x02_P2.00mm_Vertical
- removed U3: ATtiny841-SSU, Package_SO:SOIC-14_3.9x8.7mm_P1.27mm
- added ATTINY841-2: ATtiny841-SSU, Package_SO:SOIC-14_3.9x8.7mm_P1.27mm, F.Cu at (217.8, 97.5)
- added C102: 1uF, Capacitor_SMD:C_0805_2012Metric, F.Cu at (86.3, 80.7)
- added C104: 22pF, Capacitor_SMD:C_0805_2012Metric, F.Cu at (76.7, 82.8)
- added C105: 22pF, Capacitor_SMD:C_0805_2012Metric, F.Cu at (76.8, 86.5)
- added C201: 100nF, Capacitor_SMD:C_0805_2012Metric, F.Cu at (217.8, 103.2)
- added C202: 1uF, Capacitor_SMD:C_0805_2012Metric, F.Cu at (217.8, 105.3)
- added C204: 22pF, Capacitor_SMD:C_0805_2012Metric, F.Cu at (227.5, 103.2)
- added C205: 22pF, Capacitor_SMD:C_0805_2012Metric, F.Cu at (227.5, 99.5)
- added CENTER1: Screw_Terminal_01x01, diyBMSv4-Leaf:MountingHole_6.5mm_Pad_Via, F.Cu at (152.5, 93.0)
- added D100: SMBJ5.0A, Diode_SMD:D_SMB, F.Cu at (92.9, 103.0)
- added D200: SMBJ5.0A, Diode_SMD:D_SMB, F.Cu at (210.0, 102.7)
- added D201: AZ432ANTR-E1, Package_TO_SOT_SMD:SOT-23, F.Cu at (225.4, 82.0)
- added D203: DUMP, LED_SMD:LED_0805_2012Metric, F.Cu at (229.5, 81.8)
- added D204: DATA, LED_SMD:LED_0805_2012Metric, F.Cu at (213.4, 79.6)
- added EXT_TEMP_1: B2B-PH-K(LF)(SN), Connector_JST:JST_PH_B2B-PH-K_1x02_P2.00mm_Vertical, F.Cu at (92.9, 82.0)
- added EXT_TEMP_2: B2B-PH-K(LF)(SN), Connector_JST:JST_PH_B2B-PH-K_1x02_P2.00mm_Vertical, F.Cu at (218.7, 82.0)
- added F100: mSMD150, Fuse:Fuse_1812_4532Metric, F.Cu at (99.7, 101.2)
- added F200: mSMD150, Fuse:Fuse_1812_4532Metric, F.Cu at (206.0, 98.4)
- added J102: AVR-ISP-6, Connector_PinHeader_2.54mm:PinHeader_2x03_P2.54mm_Vertical, F.Cu at (88.5, 95.8)
- added J202: AVR-ISP-6, Connector_PinHeader_2.54mm:PinHeader_2x03_P2.54mm_Vertical, F.Cu at (215.6, 90.2)
- added Q201: SM2320NSAC-TRG, Package_TO_SOT_SMD:SOT-23, F.Cu at (230.4, 92.7)
- added R108: 10K, Resistor_SMD:R_0805_2012Metric, F.Cu at (92.5, 95.9)
- added R110: 3.3OHM 3/4W, Resistor_SMD:R_2010_5025Metric, F.Cu at (49.1, 84.3)
- added R111: 3.3OHM 3/4W, Resistor_SMD:R_2010_5025Metric, F.Cu at (57.7, 84.1)
- added R112: 3.3OHM 3/4W, Resistor_SMD:R_2010_5025Metric, F.Cu at (65.9, 84.1)
- added R113: 3.3OHM 3/4W, Resistor_SMD:R_2010_5025Metric, F.Cu at (49.4, 93.1)
- added R114: 3.3OHM 3/4W, Resistor_SMD:R_2010_5025Metric, F.Cu at (57.6, 93.1)
- added R115: 3.3OHM 3/4W, Resistor_SMD:R_2010_5025Metric, F.Cu at (66.0, 93.2)
- added R116: 3.3OHM 3/4W, Resistor_SMD:R_2010_5025Metric, F.Cu at (49.3, 102.3)
- added R117: 3.3OHM 3/4W, Resistor_SMD:R_2010_5025Metric, F.Cu at (58.0, 102.3)
- added R118: 3.3OHM 3/4W, Resistor_SMD:R_2010_5025Metric, F.Cu at (65.9, 102.2)
- added R121: 220, Resistor_SMD:R_0805_2012Metric, F.Cu at (93.2, 88.4)
- added R122: 4K7, Resistor_SMD:R_0805_2012Metric, F.Cu at (100.7, 80.9)
- added R201: 10K, Resistor_SMD:R_0805_2012Metric, F.Cu at (224.2, 86.4)
- added R202: CMFB103F3950FANT, Resistor_SMD:R_0805_2012Metric, F.Cu at (246.8, 88.6)
- added R203: 10K, Resistor_SMD:R_0805_2012Metric, F.Cu at (211.3, 87.6)
- added R204: 1K, Resistor_SMD:R_0805_2012Metric, F.Cu at (226.4, 86.5)
- added R205: 6.8K, Resistor_SMD:R_0805_2012Metric, F.Cu at (224.4, 92.2)
- added R206: 2.7K, Resistor_SMD:R_0805_2012Metric, F.Cu at (223.4, 96.1)
- added R207: 2K2, Resistor_SMD:R_0805_2012Metric, F.Cu at (209.9, 79.6)
- added R208: 10K, Resistor_SMD:R_0805_2012Metric, F.Cu at (211.3, 89.6)
- added R209: 2K2, Resistor_SMD:R_0805_2012Metric, F.Cu at (229.5, 85.3)
- added R210: 3.3OHM 3/4W, Resistor_SMD:R_2010_5025Metric, F.Cu at (254.5, 83.3)
- added R211: 3.3OHM 3/4W, Resistor_SMD:R_2010_5025Metric, F.Cu at (246.5, 83.3)
- added R212: 3.3OHM 3/4W, Resistor_SMD:R_2010_5025Metric, F.Cu at (238.3, 83.4)
- added R213: 3.3OHM 3/4W, Resistor_SMD:R_2010_5025Metric, F.Cu at (254.5, 92.7)
- added R214: 3.3OHM 3/4W, Resistor_SMD:R_2010_5025Metric, F.Cu at (246.4, 92.7)
- added R215: 3.3OHM 3/4W, Resistor_SMD:R_2010_5025Metric, F.Cu at (238.4, 92.7)
- added R216: 3.3OHM 3/4W, Resistor_SMD:R_2010_5025Metric, F.Cu at (254.6, 102.2)
- added R217: 3.3OHM 3/4W, Resistor_SMD:R_2010_5025Metric, F.Cu at (246.5, 102.2)
- added R218: 3.3OHM 3/4W, Resistor_SMD:R_2010_5025Metric, F.Cu at (238.4, 102.2)
- added R219: 510R, Resistor_SMD:R_0805_2012Metric, F.Cu at (227.5, 90.5)
- added R220: 10K, Resistor_SMD:R_0805_2012Metric, F.Cu at (227.5, 94.0)
- added R221: 220, Resistor_SMD:R_0805_2012Metric, F.Cu at (208.3, 88.1)
- added R222: 4K7, Resistor_SMD:R_0805_2012Metric, F.Cu at (211.3, 85.6)
- added RX1: B2B-PH-K(LF)(SN), Connector_JST:JST_PH_B2B-PH-K_1x02_P2.00mm_Vertical, F.Cu at (205.0, 92.1)
- added TX1: B2B-PH-K(LF)(SN), Connector_JST:JST_PH_B2B-PH-K_1x02_P2.00mm_Vertical, F.Cu at (100.3, 94.0)
- added Y101: 8MHZ Ceramic Resonator, Crystal:Crystal_SMD_5032-2Pin_5.0x3.2mm, F.Cu at (80.4, 84.7)
- added Y201: 8MHZ Ceramic Resonator, Crystal:Crystal_SMD_5032-2Pin_5.0x3.2mm, F.Cu at (223.8, 101.0)
- C101: renamed from C1; footprint Capacitor_SMD:C_0805_2012Metric_Pad1.15x1.40mm_HandSolder -> Capacitor_SMD:C_0805_2012Metric
- D103: renamed from D4; value RED LED -> DUMP; footprint LED_SMD:LED_0805_2012Metric_Pad1.15x1.40mm_HandSolder -> LED_SMD:LED_0805_2012Metric
- D104: renamed from D3; value Blue -> DATA; footprint LED_SMD:LED_0805_2012Metric_Pad1.15x1.40mm_HandSolder -> LED_SMD:LED_0805_2012Metric
- Q101: renamed from Q1; value IRLML6244TRPBF -> SM2320NSAC-TRG
- R101: renamed from R1; footprint Resistor_SMD:R_0805_2012Metric_Pad1.15x1.40mm_HandSolder -> Resistor_SMD:R_0805_2012Metric
- R102: renamed from R2; value NCP21WB473J03RA -> CMFB103F3950FANT; footprint Resistors_SMD:R_0603_HandSoldering -> Resistor_SMD:R_0805_2012Metric
- R103: renamed from R3; value 47K -> 10K; footprint Resistor_SMD:R_0805_2012Metric_Pad1.15x1.40mm_HandSolder -> Resistor_SMD:R_0805_2012Metric
- R104: renamed from R4; footprint Resistor_SMD:R_0805_2012Metric_Pad1.15x1.40mm_HandSolder -> Resistor_SMD:R_0805_2012Metric
- R105: renamed from R5; value 68K -> 6.8K; footprint Resistor_SMD:R_0805_2012Metric_Pad1.15x1.40mm_HandSolder -> Resistor_SMD:R_0805_2012Metric
- R106: renamed from R6; value 27K -> 2.7K; footprint Resistor_SMD:R_0805_2012Metric_Pad1.15x1.40mm_HandSolder -> Resistor_SMD:R_0805_2012Metric
- R107: renamed from R9; footprint Resistor_SMD:R_0805_2012Metric_Pad1.15x1.40mm_HandSolder -> Resistor_SMD:R_0805_2012Metric
- R109: renamed from R22; footprint Resistor_SMD:R_0805_2012Metric_Pad1.15x1.40mm_HandSolder -> Resistor_SMD:R_0805_2012Metric
- R119: renamed from R13; footprint Resistor_SMD:R_0805_2012Metric_Pad1.15x1.40mm_HandSolder -> Resistor_SMD:R_0805_2012Metric
- R120: renamed from R19; value 47K -> 10K; footprint Resistor_SMD:R_0805_2012Metric_Pad1.15x1.40mm_HandSolder -> Resistor_SMD:R_0805_2012Metric
- moved R103 21.7 mm to (92.5, 98.1), turned to 0 degrees
- moved R101 14.6 mm to (79.4, 99.3), turned to 90 degrees
- moved U2 8.18 mm to (99.2, 89.0), turned to 0 degrees
- moved Q101 4.30 mm to (73.6, 93.3)
- moved R120 3.85 mm to (76.6, 92.0)
- moved R109 3.61 mm to (74.6, 100.8)
- moved D104 3.49 mm to (83.1, 103.9), turned to 180 degrees
- moved R102 3.26 mm to (57.4, 88.8), turned to -90 degrees
- moved R104 2.95 mm to (94.6, 86.4), turned to 0 degrees
- moved R119 2.65 mm to (76.6, 95.5)
- moved D103 2.58 mm to (73.2, 106.1), turned to 180 degrees
- moved R107 2.31 mm to (86.9, 103.9), turned to 180 degrees
- moved R106 2.20 mm to (80.9, 89.7)
- moved D101 1.97 mm to (99.5, 85.2), turned to 0 degrees
- moved C101 1.85 mm to (86.3, 82.8)
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- renumbered U1 to ATTINY841-1, D1 to D101
Connections:
- net 2_VOLT renamed VREF1
- net ENABLE renamed ENABLE1
- net Net-(J1-Pad3) renamed SCK1
- +POS1 pad 1: VCC -> Net-(+POS1-Pad1)
- -NEG1 pad 1: GNDS -> Net-(-NEG1-Pad1)
- ATTINY841-1 pad 1: VCC -> +VDC
- ATTINY841-1 pad 10: DUMP_LOAD_ENABLE -> Net-(ATTINY841-1-Pad10)
- ATTINY841-1 pad 11: RXD0 -> RXD1
- ATTINY841-1 pad 12: TXD0 -> TXD1
- ATTINY841-1 pad 5: Net-(R5-Pad2) -> DUMP_LOAD_ENABLE1
- ATTINY841-1 pad 7: Net-(D2-Pad2) -> Net-(ATTINY841-1-Pad7)
- ATTINY841-1 pad 8: Net-(D3-Pad2) -> MISO1
- C101 pad 1: VCC -> +VDC
- D103 pad 2: VCC -> +VDC
- D104 pad 2: Net-(D3-Pad2) -> Net-(ATTINY841-1-Pad7)
- R101 pad 1: VCC -> +VDC
- R105 pad 2: Net-(R5-Pad2) -> Net-(ATTINY841-1-Pad10)
- R106 pad 1: Net-(R5-Pad2) -> Net-(ATTINY841-1-Pad10)
- R119 pad 2: DUMP_LOAD_ENABLE -> DUMP_LOAD_ENABLE1
- U4 pad 2: GNDS -> -VDC
- U4 pad 3: RXD0 -> RXD1
- U4 pad 4: VCC -> +VDC
Routing:
- net VCC: track 132.3 -> 0.00 mm, vias 42 -> 0
- net RXD0: track 126.3 -> 0.00 mm, vias 2 -> 0
- net +VDC: track 18.7 -> 109.5 mm, vias 0 -> 47
- net RXD1: track 49.1 -> 125.1 mm
- net VREF2: track 0.00 -> 57.4 mm, vias 0 -> 3
- net Net-(J3-Pad3): track 54.9 -> 0.00 mm, vias 2 -> 0
- net SCK2: track 0.00 -> 52.0 mm, vias 0 -> 2
- net 2_VOLT_1: track 50.6 -> 0.00 mm, vias 3 -> 0
- net Net-(TX1-Pad1): track 37.4 -> 4.16 mm
- net Net-(TX1-Pad2): track 34.5 -> 6.20 mm
- net -VDC: track 0.00 -> 27.6 mm, vias 0 -> 29
- net DUMP_LOAD_ENABLE: track 25.2 -> 0.00 mm, vias 2 -> 0
- net MISO1: track 0.00 -> 23.2 mm
- net RXD2: track 0.00 -> 21.2 mm, vias 0 -> 1
- net DUMP_LOAD_ENABLE_1: track 20.8 -> 0.00 mm, vias 2 -> 0
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- added copper zone on B.Cu, net +VDC
- added copper zone on B.Cu, net -VDC
- added copper zone on F.Cu, net -VDC
- added copper zone on B.Cu, net Net-(+POS1-Pad1)
- added copper zone on F.Cu, net Net-(+POS1-Pad1)
- added copper zone on B.Cu, net Net-(-NEG1-Pad1)
- added copper zone on F.Cu, net Net-(-NEG1-Pad1)
- added copper zone on F.Cu, net Net-(Q201-Pad3)
- added copper zone on F.Cu, net Net-(R110-Pad2)
- added copper zone on F.Cu, net Net-(R111-Pad2)
- added copper zone on F.Cu, net Net-(R210-Pad2)
- added copper zone on F.Cu, net Net-(R211-Pad2)
- removed copper zone on B.Cu, net GNDS
- removed copper zone on F.Cu, net GNDS
- removed copper zone on F.Cu, net Net-(Q2-Pad3)
- removed copper zone on B.Cu, net VCC
- removed copper zone on F.Cu, net VCC
Other:
- outline, holes or cut-outs redrawn
- net class Default removed
- board text added: "BMS for LEAF Module v2.01 - Joho Technology Inc. 2021 Based on diy BMS version 4 for Nissan Leaf cells by Stuart Pittaway."
- board text added: "v2.01 Joho Technology Inc. 2021"
- board text removed: "v1.00"
