File: diyBMSv4-Leaf_neg.kicad_sch (KiCad schematic)
At the start: 39 parts, among them J202 AVR-ISP-6, Q201 SM2320NSAC-TRG, Y201 8MHZ Ceramic Resonator

Commit message: V2.0.1
Parts:
- removed R206, R207, R209, R210, R222, R224, R225, R226, R227, R228, R229, R230: 3.3OHM 3/4W, Resistor_SMD:R_1210_3225Metric, symbol Device:R
- added R214, R215, R216, R217, R218: 3.3OHM 3/4W, Resistor_SMD:R_2010_5025Metric, symbol Device:R
- R210: renamed from R208; footprint Resistor_SMD:R_1210_3225Metric -> Resistor_SMD:R_2010_5025Metric; LCSCStockCode C21624 -> C270971; PartNumber 1210W3F330KT5E -> 201007F330KT4E
- R211, R212, R213: footprint Resistor_SMD:R_1210_3225Metric -> Resistor_SMD:R_2010_5025Metric; LCSCStockCode C21624 -> C270971; PartNumber 1210W3F330KT5E -> 201007F330KT4E
- renumbered R219 to R202, R220 to R203, R202 to R204, R203 to R205, R204 to R206, R218 to R207, R221 to R208, R217 to R209, R214 to R219, R215 to R220
Connections:
- net GND: now also R210.1, R213.1, R216.1
- net at Q201.3 (D), R209.1, R212.2: now also R215.2, R218.2; no longer R213.2
- net at R210.2, R211.1: now also R213.2, R214.1, R216.2, R217.1
- net at R211.2, R212.1: now also R214.2, R215.1, R217.2, R218.1; no longer R213.1
Other:
- note added: "CHIP RESISTOR - SURFACE MOUNT 3.3OHMS ±1% 3/4W 2010 ROHS, 3 in series with 3 in parallel gives 3.30 Ohm equivalent resistance 9 resistors provide 9*0.75W=6.75W of power disipation. Balance current (at 3.3ohm): 1.27A at 4.2V and 5.35W power 1.21A at 4.0V and 4.84W power 1.13A at 3.75V and 4.26W power"
- note removed: "CHIP RESISTOR - SURFACE MOUNT 3.3OHMS ±1% 3/4W 1210 ROHS, 4 in series with 4 in parallel gives 3.30 Ohm equivalent resistance 16 resistors provide 16*0.75W=12W of power dissipation. Balance current: 1.27A at 4.2V and 5.35W power 1.21A at 4.0V and 4.84W power 1.13A at 3.75V and 4.26W power"
