File: diyBMSv4-Leaf_pos.kicad_sch (KiCad schematic)
At the start: 39 parts, among them J102 AVR-ISP-6, Q101 SM2320NSAC-TRG, Y101 8MHZ Ceramic Resonator

Commit message: V2.0.1
Parts:
- removed R106, R107, R109, R110, R122, R124, R125, R126, R127, R128, R129, R130: 3.3OHM 3/4W, Resistor_SMD:R_1210_3225Metric, symbol Device:R
- added R114, R115, R116, R117, R118: 3.3OHM 3/4W, Resistor_SMD:R_2010_5025Metric, symbol Device:R
- R110: renamed from R108; footprint Resistor_SMD:R_1210_3225Metric -> Resistor_SMD:R_2010_5025Metric; JLCPCBRotation 0 -> (none); LCSCStockCode C21624 -> C270971; PartNumber 1210W3F330KT5E -> 201007F330KT4E
- R111, R112, R113: footprint Resistor_SMD:R_1210_3225Metric -> Resistor_SMD:R_2010_5025Metric; JLCPCBRotation 0 -> (none); LCSCStockCode C21624 -> C270971; PartNumber 1210W3F330KT5E -> 201007F330KT4E
- renumbered R119 to R102, R120 to R103, R102 to R104, R103 to R105, R104 to R106, R118 to R107, R121 to R108, R117 to R109, R114 to R119, R115 to R120
Connections:
- net +VDC: now also R110.1, R113.1, R116.1
- net at Q101.3 (D), R109.1, R112.2: now also R115.2, R118.2; no longer R113.2
- net at R110.2, R111.1: now also R113.2, R114.1, R116.2, R117.1
- net at R111.2, R112.1: now also R114.2, R115.1, R117.2, R118.1; no longer R113.1
Other:
- note added: "CHIP RESISTOR - SURFACE MOUNT 3.3OHMS ±1% 3/4W 2010 ROHS, 3 in series with 3 in parallel gives 3.30 Ohm equivalent resistance 9 resistors provide 9*0.75W=6.75W of power disipation. Balance current (at 3.3ohm): 1.27A at 4.2V and 5.35W power 1.21A at 4.0V and 4.84W power 1.13A at 3.75V and 4.26W power"
- note removed: "CHIP RESISTOR - SURFACE MOUNT 3.3OHMS ±1% 3/4W 1210 ROHS, 4 in series with 4 in parallel gives 3.30 Ohm equivalent resistance 16 resistors provide 16*0.75W=12W of power dissipation. Balance current: 1.27A at 4.2V and 5.35W power 1.21A at 4.0V and 4.84W power 1.13A at 3.75V and 4.26W power"
