File: file5DF129FA.kicad_sch (KiCad schematic)
At the start: 15 parts, among them U2 EL3H7(B)(TA)-G, U4 EL3H7(B)(TA)-G

Commit message: V2.0.1
Parts:
- renumbered R105 to R121, R116 to R122, R205 to R221, R216 to R222
Other:
- note added: "::::NOTE:::: Once the 2pin connectors are soldered trim the legs as flush with the solder as possible."
- note added: "The Leaf cell is 2s2P with 3 connection terminals, +ve common -ve Voltage on one pack is measured between the -ve terminal and common. The voltage on the second pack measures between the +ve terminal and common. Each BMS is has its own supply: +ve terminal - common (common is negative) -ve terminal - common ( common is positive)"
- note removed: "::::NOTE:::: Once the 2pin and 4 pin connectors are soldered trim the legs as flush with the solder as possible,"
- note removed: "The Leaf cell is 2s2P with 3 connection terminals, +ve common -ve Voltage on one pack is measured between the -ve terminal and common. The voltage on the second pack measures between he +ve terminal and common. For schematic and layout purposes there are uniquely names VCC lines and GND lines for the separated BMS circuits. YES... confusing Each BMS is has its own supply: +ve terminal - common (c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"
Changed lines of the file:
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@@
   (title_block
     (title "diyBMSv4 - LEAF")
-    (date "2021-03-07")
-    (rev "2.00")
+    (date "2021-03-10")
+    (rev "2.01")
     (company "Joho Technology Inc")
   )
@@
     (stroke (width 0) (type dash) (color 0 0 0 0))
   )
-  (text "The Leaf cell is 2s2P with 3 connection terminals,  +ve  common -ve\nVoltage on one pack is measured between the -ve terminal and\ncommon. The voltage on the second pack measures between he +ve\nterminal and common.\nFor schematic and layout purposes there are uniquely names VCC\nlines and GND lines for the separated BMS circuits.\nYES... confusing\n\nEach BMS is has its own supply:\n +ve terminal - common  (common is negative)\n -ve terminal - common ( common is positive)"
+  (text "The Leaf cell is 2s2P with 3 connection terminals,  +ve  common -ve\nVoltage on one pack is measured between the -ve terminal and\ncommon. The voltage on the second pack measures between the +ve\nterminal and common.\n\nEach BMS is has its own supply:\n +ve terminal - common  (common is negative)\n -ve terminal - common ( common is positive)"
     (at 26.924 193.675 0)
     (effects (font (size 2.54 2.54)) (justify left bottom))
@@
     (effects (font (size 5.08 5.08)) (justify left bottom))
   )
-  (text "::::NOTE::::\nOnce the 2pin and 4 pin connectors\nare soldered trim the legs as flush with the\nsolder as possible,"
+  (text "::::NOTE::::\nOnce the 2pin connectors\nare soldered trim the legs as flush with the\nsolder as possible."
     (at 205.232 101.854 0)
     (effects (font (size 1.27 1.27) (thickness 0.254) bold) (justify left bottom))
@@
   (symbol (lib_id "diyBMS-Leaf-rescue:R-Device") (at 80.772 78.74 270) (unit 1)
     (in_bom yes) (on_board yes)
-    (property "Reference" "R105" (id 0) (at 80.772 73.4822 90))
+    (property "Reference" "R121" (id 0) (at 80.772 73.482 90))
     (property "Value" "220" (id 1) (at 80.772 75.7936 90))
     (property "Footprint" "Resistor_SMD:R_0805_2012Metric" (id 2) (at 80.772 76.962 90)
@@
   (symbol (lib_id "diyBMS-Leaf-rescue:R-Device") (at 132.334 55.626 180) (unit 1)
     (in_bom yes) (on_board yes)
-    (property "Reference" "R116" (id 0) (at 137.592 55.626 90))
+    (property "Reference" "R122" (id 0) (at 137.592 55.626 90))
     (property "Value" "4K7" (id 1) (at 135.2804 55.626 90))
     (property "Footprint" "Resistor_SMD:R_0805_2012Metric" (id 2) (at 134.112 55.626 90)
@@
   (symbol (lib_id "diyBMS-Leaf-rescue:R-Device") (at 168.91 46.355 270) (unit 1)
     (in_bom yes) (on_board yes)
-    (property "Reference" "R205" (id 0) (at 168.91 41.097 90))
+    (property "Reference" "R221" (id 0) (at 168.91 41.097 90))
     (property "Value" "220" (id 1) (at 168.91 43.4086 90))
     (property "Footprint" "Resistor_SMD:R_0805_2012Metric" (id 2) (at 168.91 44.577 90)
@@
   (symbol (lib_id "diyBMS-Leaf-rescue:R-Device") (at 191.135 94.615 180) (unit 1)
     (in_bom yes) (on_board yes)
-    (property "Reference" "R216" (id 0) (at 196.393 94.615 90))
+    (property "Reference" "R222" (id 0) (at 196.393 94.615 90))
     (property "Value" "4K7" (id 1) (at 194.0814 94.615 90))
     (property "Footprint" "Resistor_SMD:R_0805_2012Metric" (id 2) (at 192.913 94.615 90)
